File: Hardware/USB 2.0 Pads.sch (KiCad schematic (older format))
At the start: 3 parts, among them J1 USB_A, P1 USB_C_Plug_USB2.0

Commit message: Updated files
Parts:
- P1: footprint SnapEDA Library:GCT_USB4155-03-C_REVA -> Expansion_Card:USB_C_Plug_Molex_105444
- R1: footprint Resistor_SMD:R_0805_2012Metric_Pad1.20x1.40mm_HandSolder -> Resistor_SMD:R_0805_2012Metric
Changed lines of the file:
@@
 F 0 "P1" H 2307 4267 50  0000 C CNN
 F 1 "USB_C_Plug_USB2.0" H 2307 4176 50  0000 C CNN
-F 2 "SnapEDA Library:GCT_USB4155-03-C_REVA" H 2350 3400 50  0001 C CNN
+F 2 "Expansion_Card:USB_C_Plug_Molex_105444" H 2350 3400 50  0001 C CNN
 F 3 "https://www.usb.org/sites/default/files/documents/usb_type-c.zip" H 2350 3400 50  0001 C CNN
 	1    2200 3400
@@
 F 0 "R1" V 2745 3000 50  0000 C CNN
 F 1 "5.1k" V 2836 3000 50  0000 C CNN
-F 2 "Resistor_SMD:R_0805_2012Metric_Pad1.20x1.40mm_HandSolder" V 2990 2990 50  0001 C CNN
+F 2 "Resistor_SMD:R_0805_2012Metric" V 2990 2990 50  0001 C CNN
 F 3 "~" H 2950 3000 50  0001 C CNN
 	1    2950 3000
